Commit message: Adjusted the initial position of joint 5 to avoid singularity error at start of moveit_servo node

File: annin_ar4_description/urdf/ar_macro.xacro (robot description, xacro)
@@ -194,5 +194,5 @@
     </link>
     <joint name="${tf_prefix}joint_5" type="revolute">
-      <origin rpy="${pi} 0 -1.5708" xyz="0 0 -0.22263"/>
+      <origin rpy="-1.57075 0 -1.57075" xyz="0 0 -0.22263"/>
       <parent link="${tf_prefix}link_4"/>
       <child link="${tf_prefix}link_5"/>
