Commit message: hardcode the ar_model variable

File: annin_ar4_description/urdf/ar.urdf.xacro (robot description, xacro)
@@ -1,4 +1,5 @@
 <?xml version="1.0"?>
-<robot xmlns:xacro="http://wiki.ros.org/xacro" name="$(arg ar_model)">
+<robot xmlns:xacro="http://wiki.ros.org/xacro" name="mk3">
+  <xacro:property name="ar_model" value="mk3" />
   <xacro:arg name="tf_prefix" default="" />
   <xacro:arg name="include_gripper" default="true" />
@@ -10,11 +11,10 @@
     <parent link="world" />
     <child link="Abb_dummy_base" />
-    <origin xyz="0 -1.110
-      0" rpy="0 0 0" />
+    <origin xyz="0 -1.110 0" rpy="0 0 0" />
   </joint>
   <xacro:ar_robot
     tf_prefix="$(arg tf_prefix)"
     parent="world"
-    robot_parameters_file="$(find annin_ar4_description)/config/$(arg ar_model).yaml"
+    robot_parameters_file="$(find annin_ar4_description)/config/${ar_model}.yaml"
   >
     <origin xyz="0 0 0" rpy="0 0 0" />

Commit message: full_system_update

File: annin_ar4_description/urdf/ar.urdf.xacro (robot description, xacro)
@@ -1,5 +1,4 @@
 <?xml version="1.0"?>
-<robot xmlns:xacro="http://wiki.ros.org/xacro" name="mk3">
-  <xacro:property name="ar_model" value="mk3" />
+<robot xmlns:xacro="http://wiki.ros.org/xacro" name="$(arg ar_model)">
   <xacro:arg name="tf_prefix" default="" />
   <xacro:arg name="include_gripper" default="true" />
@@ -7,22 +6,16 @@
   <xacro:include filename="$(find annin_ar4_description)/urdf/ar_gripper_macro.xacro" />
   <link name="world" />
-  <link name="Abb_dummy_base" />
-  <joint name="ABB_base_joint" type="fixed">
+  <link name="ABB_base_link" />
+  <joint name="ABB_base_link_to_world_joint" type="fixed">
     <parent link="world" />
-    <child link="Abb_dummy_base" />
-    <origin xyz="0 -1.110 0" rpy="0 0 0" />
+    <child link="ABB_base_link" />
+    <origin xyz="0 -1.110
+      0" rpy="0 0 1.57079" />
   </joint>
-  <xacro:ar_robot
-    tf_prefix="$(arg tf_prefix)"
-    parent="world"
-    robot_parameters_file="$(find annin_ar4_description)/config/${ar_model}.yaml"
-  >
+  <xacro:ar_robot tf_prefix="$(arg tf_prefix)" parent="world" robot_parameters_file="$(find annin_ar4_description)/config/$(arg ar_model).yaml">
     <origin xyz="0 0 0" rpy="0 0 0" />
   </xacro:ar_robot>
   <xacro:if value="$(arg include_gripper)">
-    <xacro:ar_gripper
-      tf_prefix="$(arg tf_prefix)"
-      parent="$(arg tf_prefix)ee_link"
-    />
+    <xacro:ar_gripper tf_prefix="$(arg tf_prefix)" parent="$(arg tf_prefix)ee_link" />
   </xacro:if>
 </robot>

File: annin_ar4_description/urdf/ar_gazebo.urdf.xacro (robot description, xacro)
@@ -9,41 +9,20 @@
   <xacro:arg name="include_gripper" default="True" />
   <link name="world" />
-  <link name="Abb_dummy_base" />
-  <joint name="ABB_base_joint" type="fixed">
+  <link name="ABB_base_link" />
+  <joint name="ABB_base_link_to_world_joint" type="fixed">
     <parent link="world" />
-    <child link="Abb_dummy_base" />
-    <origin xyz="0 -1.110  0" rpy="0 0 0" />
+    <child link="ABB_base_link" />
+    <origin xyz="0 -1.110
+      0" rpy="0 0 0" />
   </joint>
-  <xacro:ar_robot
-    tf_prefix="$(arg tf_prefix)"
-    parent="world"
-    robot_parameters_file="$(find annin_ar4_description)/config/$(arg ar_model).yaml"
-  >
+  <xacro:ar_robot tf_prefix="$(arg tf_prefix)" parent="world" robot_parameters_file="$(find annin_ar4_description)/config/$(arg ar_model).yaml">
     <origin xyz="0 0 0" rpy="0 0 0" />
   </xacro:ar_robot>
   <xacro:if value="$(arg include_gripper)">
     <xacro:include filename="$(find annin_ar4_description)/urdf/ar_gripper_macro.xacro" />
-    <xacro:ar_gripper
-      tf_prefix="$(arg tf_prefix)"
-      parent="$(arg tf_prefix)ee_link"
-    />
-    <xacro:ar_gripper_ros2_control
-      name="ARGripperGazeboSystem"
-      plugin_name="gz_ros2_control/GazeboSimSystem"
-      serial_port="None"
-      driver_parameters_file="$(find annin_ar4_driver)/config/gripper_driver.yaml"
-      tf_prefix="$(arg tf_prefix)"
-    />
+    <xacro:ar_gripper tf_prefix="$(arg tf_prefix)" parent="$(arg tf_prefix)ee_link" />
+    <xacro:ar_gripper_ros2_control name="ARGripperGazeboSystem" plugin_name="gz_ros2_control/GazeboSimSystem" serial_port="None" driver_parameters_file="$(find annin_ar4_driver)/config/gripper_driver.yaml" tf_prefix="$(arg tf_prefix)" />
   </xacro:if>
-  <xacro:ar_ros2_control
-    ar_model="$(arg ar_model)"
-    plugin_name="gz_ros2_control/GazeboSimSystem"
-    serial_port="None"
-    calibrate="False"
-    robot_parameters_file="$(find annin_ar4_description)/config/$(arg ar_model).yaml"
-    joint_offset_parameters_file="$(find annin_ar4_driver)/config/joint_offsets/$(arg ar_model).yaml"
-    driver_parameters_file="$(find annin_ar4_driver)/config/driver.yaml"
-    tf_prefix="$(arg tf_prefix)"
-  />
+  <xacro:ar_ros2_control ar_model="$(arg ar_model)" plugin_name="gz_ros2_control/GazeboSimSystem" serial_port="None" calibrate="False" robot_parameters_file="$(find annin_ar4_description)/config/$(arg ar_model).yaml" joint_offset_parameters_file="$(find annin_ar4_driver)/config/joint_offsets/$(arg ar_model).yaml" driver_parameters_file="$(find annin_ar4_driver)/config/driver.yaml" tf_prefix="$(arg tf_prefix)" />
   <gazebo reference="world" />
   <gazebo>

File: annin_ar4_description/urdf/ar_gripper_macro.xacro (robot description, xacro)
@@ -14,41 +14,23 @@
       <child link="${tf_prefix}gripper_base_link" />
     </joint>
-    <link
-      name="${tf_prefix}gripper_base_link">
+    <link name="${tf_prefix}gripper_base_link">
       <inertial>
-        <origin
-          xyz="0.000218865638025569 -5.75810071732045E-05 0.0188189080442559"
-          rpy="0 0 0" />
-        <mass
-          value="0.0779213197542101" />
-        <inertia
-          ixx="1.27018244320936E-05"
-          ixy="-1.98293669536147E-07"
-          ixz="-2.58632439119383E-07"
-          iyy="2.84792796640278E-05"
-          iyz="-4.25276765641554E-07"
-          izz="3.57075748419373E-05" />
+        <origin xyz="0.000218865638025569 -5.75810071732045E-05 0.0188189080442559" rpy="0 0 0" />
+        <mass value="0.0779213197542101" />
+        <inertia ixx="1.27018244320936E-05" ixy="-1.98293669536147E-07" ixz="-2.58632439119383E-07" iyy="2.84792796640278E-05" iyz="-4.25276765641554E-07" izz="3.57075748419373E-05" />
       </inertial>
       <visual>
-        <origin
-          xyz="0 0 0"
-          rpy="0 0 0" />
+        <origin xyz="0 0 0" rpy="0 0 0" />
         <geometry>
-          <mesh
-            filename="file://$(find annin_ar4_description)/meshes/ar4_gripper/gripper_base_link.stl" />
+          <mesh filename="file://$(find annin_ar4_description)/meshes/ar4_gripper/gripper_base_link.stl" />
         </geometry>
-        <material
-          name="">
-          <color
-            rgba="0.792156862745098 0.819607843137255 0.933333333333333 1" />
+        <material name="">
+          <color rgba="0.792156862745098 0.819607843137255 0.933333333333333 1" />
         </material>
       </visual>
       <collision>
-        <origin
-          xyz="0 0 0"
-          rpy="0 0 0" />
+        <origin xyz="0 0 0" rpy="0 0 0" />
         <geometry>
-          <mesh
-            filename="file://$(find annin_ar4_description)/meshes/ar4_gripper/gripper_base_link.stl" />
+          <mesh filename="file://$(find annin_ar4_description)/meshes/ar4_gripper/gripper_base_link.stl" />
         </geometry>
       </collision>
@@ -56,38 +38,21 @@
     <link name="${tf_prefix}gripper_jaw1_link">
       <inertial>
-        <origin
-          xyz="0.0068393 0.0018263 -0.0052235"
-          rpy="0 0 0" />
-        <mass
-          value="0.0080032" />
-        <inertia
-          ixx="7.6628E-07"
-          ixy="2.1048E-07"
-          ixz="4.3688E-09"
-          iyy="1.0775E-06"
-          iyz="-7.4587E-08"
-          izz="1.3907E-06" />
+        <origin xyz="0.0068393 0.0018263 -0.0052235" rpy="0 0 0" />
+        <mass value="0.0080032" />
+        <inertia ixx="7.6628E-07" ixy="2.1048E-07" ixz="4.3688E-09" iyy="1.0775E-06" iyz="-7.4587E-08" izz="1.3907E-06" />
       </inertial>
       <visual>
-        <origin
-          xyz="0 0 0"
-          rpy="0 0 0" />
+        <origin xyz="0 0 0" rpy="0 0 0" />
         <geometry>
-          <mesh
-            filename="file://$(find annin_ar4_description)/meshes/ar4_gripper/gripper_jaw1_link.stl" />
+          <mesh filename="file://$(find annin_ar4_description)/meshes/ar4_gripper/gripper_jaw1_link.stl" />
         </geometry>
-        <material
-          name="">
-          <color
-            rgba="1 1 1 1" />
+        <material name="">
+          <color rgba="1 1 1 1" />
         </material>
       </visual>
       <collision>
-        <origin
-          xyz="0 0 0"
-          rpy="0 0 0" />
+        <origin xyz="0 0 0" rpy="0 0 0" />
         <geometry>
-          <mesh
-            filename="file://$(find annin_ar4_description)/meshes/ar4_gripper/gripper_jaw1_link.stl" />
+          <mesh filename="file://$(find annin_ar4_description)/meshes/ar4_gripper/gripper_jaw1_link.stl" />
         </geometry>
       </collision>
@@ -95,72 +60,38 @@
     <link name="${tf_prefix}gripper_jaw2_link">
       <inertial>
-        <origin
-          xyz="0.0068393 0.0018263 -0.0052235"
-          rpy="0 0 0" />
-        <mass
-          value="0.0080032" />
-        <inertia
-          ixx="7.6628E-07"
-          ixy="2.1048E-07"
-          ixz="4.3688E-09"
-          iyy="1.0775E-06"
-          iyz="-7.4587E-08"
-          izz="1.3907E-06" />
+        <origin xyz="0.0068393 0.0018263 -0.0052235" rpy="0 0 0" />
+        <mass value="0.0080032" />
+        <inertia ixx="7.6628E-07" ixy="2.1048E-07" ixz="4.3688E-09" iyy="1.0775E-06" iyz="-7.4587E-08" izz="1.3907E-06" />
       </inertial>
       <visual>
-        <origin
-          xyz="0 0 0"
-          rpy="0 0 0" />
+        <origin xyz="0 0 0" rpy="0 0 0" />
         <geometry>
-          <mesh
-            filename="file://$(find annin_ar4_description)/meshes/ar4_gripper/gripper_jaw2_link.stl" />
+          <mesh filename="file://$(find annin_ar4_description)/meshes/ar4_gripper/gripper_jaw2_link.stl" />
         </geometry>
-        <material
-          name="">
-          <color
-            rgba="1 1 1 1" />
+        <material name="">
+          <color rgba="1 1 1 1" />
         </material>
       </visual>
       <collision>
-        <origin
-          xyz="0 0 0"
-          rpy="0 0 0" />
+        <origin xyz="0 0 0" rpy="0 0 0" />
         <geometry>
-          <mesh
-            filename="file://$(find annin_ar4_description)/meshes/ar4_gripper/gripper_jaw2_link.stl" />
+          <mesh filename="file://$(find annin_ar4_description)/meshes/ar4_gripper/gripper_jaw2_link.stl" />
         </geometry>
       </collision>
     </link>
     <joint name="${tf_prefix}gripper_jaw1_joint" type="prismatic">
-      <origin
-        xyz="0.014 -0.0029 0.001"
-        rpy="1.5708 0 0 " />
-      <parent
-        link="${tf_prefix}gripper_base_link" />
-      <child
-        link="${tf_prefix}gripper_jaw1_link" />
-      <axis
-        xyz="-1 0 0" />
-      <limit
-        lower="0"
-        upper="0.015"
-        effort="1000"
-        velocity="1.0" />
+      <origin xyz="0.014 -0.0029 0.001" rpy="1.5708 0 0 " />
+      <parent link="${tf_prefix}gripper_base_link" />
+      <child link="${tf_prefix}gripper_jaw1_link" />
+      <axis xyz="-1 0 0" />
+      <limit lower="0" upper="0.015" effort="1000" velocity="1.0" />
     </joint>
     <joint name="${tf_prefix}gripper_jaw2_joint" type="prismatic">
-      <origin
-        xyz="-0.014 -0.0029 0.001"
-        rpy="1.5708 0 0" />
-      <parent
-        link="${tf_prefix}gripper_base_link" />
-      <child
-        link="${tf_prefix}gripper_jaw2_link" />
-      <axis
-        xyz="1 0 0" />
-      <limit
-        lower="0"
-        upper="0.015"
-        effort="1000"
-        velocity="1.0" />
+      <origin xyz="-0.014 -0.0029 0.001" rpy="1.5708 0 0" />
+      <parent link="${tf_prefix}gripper_base_link" />
+      <child link="${tf_prefix}gripper_jaw2_link" />
+      <axis xyz="1 0 0" />
+      <limit lower="0" upper="0.015" effort="1000" velocity="1.0" />
+      <mimic joint="${tf_prefix}gripper_jaw1_joint" multiplier="1"/>
     </joint>
   </xacro:macro>

File: annin_ar4_description/urdf/ar_macro.xacro (robot description, xacro)
@@ -194,5 +194,5 @@
     </link>
     <joint name="${tf_prefix}joint_5" type="revolute">
-      <origin rpy="-1.57075 0 -1.57075" xyz="0 0 -0.22263"/>
+      <origin rpy="${pi} 0 -1.57075" xyz="0 0 -0.22263"/>
       <parent link="${tf_prefix}link_4"/>
       <child link="${tf_prefix}link_5"/>

File: annin_ar4_driver/urdf/ar.urdf.xacro (robot description, xacro)
@@ -10,11 +10,10 @@
   <xacro:include filename="$(find annin_ar4_description)/urdf/ar_gripper.ros2_control.xacro" />
   <xacro:include filename="$(find annin_ar4_description)/urdf/ar_gripper_macro.xacro" />
-  <xacro:include filename="$(find annin_ar4_description)/urdf/ar_camera_macro.xacro" />
   <link name="world" />
-  <link name="Abb_dummy_base" />
+  <link name="ABB_base_link" />
   <joint name="ABB_base_joint" type="fixed">
     <parent link="world" />
-    <child link="Abb_dummy_base" />
-    <origin xyz="0 -1.110  0" rpy="0 0 0" />
+    <child link="ABB_base_link" />
+    <origin xyz="0 -1.110  0" rpy="0 0 1.57079" />
   </joint>
   <xacro:ar_robot
@@ -35,8 +34,4 @@
     tf_prefix="$(arg tf_prefix)"
   />
-  <xacro:ar_camera
-      tf_prefix="$(arg tf_prefix)"
-      parent="$(arg tf_prefix)ee_link"
-    />
   <xacro:if value="$(arg include_gripper)">
     <xacro:ar_gripper

File: annin_ar4_moveit_config/srdf/ar_macro.srdf.xacro (robot description, xacro)
@@ -22,5 +22,5 @@
       <joint name="${tf_prefix}joint_3" value="0" />
       <joint name="${tf_prefix}joint_4" value="0" />
-      <joint name="${tf_prefix}joint_5" value="0" />
+      <joint name="${tf_prefix}joint_5" value="1.5707" />
       <joint name="${tf_prefix}joint_6" value="0" />
     </group_state>
