Commit message: new AR4 driver: Added new AR4 driver

File: annin_ar4_description/urdf/ar.urdf.xacro (robot description, xacro)
@@ -4,6 +4,4 @@
   <xacro:arg name="include_gripper" default="true" />
   <xacro:include filename="$(find annin_ar4_description)/urdf/ar_macro.xacro" />
-  <xacro:include filename="$(find annin_ar4_description)/urdf/ar_gripper_macro.xacro" />
-  <link name="world" />
   <link name="ABB_base_link" />
   <joint name="ABB_base_link_to_world_joint" type="fixed">
@@ -13,9 +11,18 @@
       0" rpy="0 0 1.57079" />
   </joint>
-  <xacro:ar_robot tf_prefix="$(arg tf_prefix)" parent="world" robot_parameters_file="$(find annin_ar4_description)/config/$(arg ar_model).yaml">
+  <link name="world" />
+  <xacro:ar_robot
+    tf_prefix="$(arg tf_prefix)"
+    parent="world"
+    robot_parameters_file="$(find annin_ar4_description)/config/$(arg ar_model).yaml"
+  >
     <origin xyz="0 0 0" rpy="0 0 0" />
   </xacro:ar_robot>
   <xacro:if value="$(arg include_gripper)">
-    <xacro:ar_gripper tf_prefix="$(arg tf_prefix)" parent="$(arg tf_prefix)ee_link" />
+    <xacro:include filename="$(find annin_ar4_description)/urdf/ar_gripper_macro.xacro" />
+    <xacro:ar_gripper
+      tf_prefix="$(arg tf_prefix)"
+      parent="$(arg tf_prefix)ee_link"
+    />
   </xacro:if>
 </robot>

File: annin_ar4_description/urdf/ar_gazebo.urdf.xacro (robot description, xacro)
@@ -2,4 +2,5 @@
 <robot xmlns:xacro="http://wiki.ros.org/xacro" name="$(arg ar_model)">
   <xacro:include filename="$(find annin_ar4_description)/urdf/ar_macro.xacro" />
+  <xacro:include filename="$(find annin_ar4_description)/urdf/ar_gripper_macro.xacro" />
   <xacro:include filename="$(find annin_ar4_description)/urdf/ar.ros2_control.xacro" />
   <xacro:include filename="$(find annin_ar4_description)/urdf/ar_gripper.ros2_control.xacro" />
@@ -7,6 +8,4 @@
   <xacro:arg name="tf_prefix" default="" />
   <xacro:arg name="namespace" default="" />
-  <xacro:arg name="include_gripper" default="True" />
-  <link name="world" />
   <link name="ABB_base_link" />
   <joint name="ABB_base_link_to_world_joint" type="fixed">
@@ -16,13 +15,33 @@
       0" rpy="0 0 1.57079" />
   </joint>
-  <xacro:ar_robot tf_prefix="$(arg tf_prefix)" parent="world" robot_parameters_file="$(find annin_ar4_description)/config/$(arg ar_model).yaml">
+  <link name="world" />
+  <xacro:ar_robot
+    tf_prefix="$(arg tf_prefix)"
+    parent="world"
+    robot_parameters_file="$(find annin_ar4_description)/config/$(arg ar_model).yaml"
+  >
     <origin xyz="0 0 0" rpy="0 0 0" />
   </xacro:ar_robot>
-  <xacro:if value="$(arg include_gripper)">
-    <xacro:include filename="$(find annin_ar4_description)/urdf/ar_gripper_macro.xacro" />
-    <xacro:ar_gripper tf_prefix="$(arg tf_prefix)" parent="$(arg tf_prefix)ee_link" />
-    <xacro:ar_gripper_ros2_control name="ARGripperGazeboSystem" plugin_name="gz_ros2_control/GazeboSimSystem" serial_port="None" driver_parameters_file="$(find annin_ar4_driver)/config/gripper_driver.yaml" tf_prefix="$(arg tf_prefix)" />
-  </xacro:if>
-  <xacro:ar_ros2_control ar_model="$(arg ar_model)" plugin_name="gz_ros2_control/GazeboSimSystem" serial_port="None" calibrate="False" robot_parameters_file="$(find annin_ar4_description)/config/$(arg ar_model).yaml" joint_offset_parameters_file="$(find annin_ar4_driver)/config/joint_offsets/$(arg ar_model).yaml" driver_parameters_file="$(find annin_ar4_driver)/config/driver.yaml" tf_prefix="$(arg tf_prefix)" />
+  <xacro:ar_gripper
+    tf_prefix="$(arg tf_prefix)"
+    parent="$(arg tf_prefix)ee_link"
+  />
+  <xacro:ar_ros2_control
+    ar_model="$(arg ar_model)"
+    plugin_name="gz_ros2_control/GazeboSimSystem"
+    serial_port="None"
+    calibrate="False"
+    robot_parameters_file="$(find annin_ar4_description)/config/$(arg ar_model).yaml"
+    joint_offset_parameters_file="$(find annin_ar4_driver)/config/joint_offsets/$(arg ar_model).yaml"
+    driver_parameters_file="$(find annin_ar4_driver)/config/driver.yaml"
+    tf_prefix="$(arg tf_prefix)"
+  />
+  <xacro:ar_gripper_ros2_control
+    name="ARGripperGazeboSystem"
+    plugin_name="gz_ros2_control/GazeboSimSystem"
+    serial_port="None"
+    driver_parameters_file="$(find annin_ar4_driver)/config/gripper_driver.yaml"
+    tf_prefix="$(arg tf_prefix)"
+  />
   <gazebo reference="world" />
   <gazebo>

File: annin_ar4_description/urdf/ar_gripper_macro.xacro (robot description, xacro)
@@ -1,7 +1,3 @@
 <?xml version="1.0" encoding="utf-8"?>
-<!-- This URDF was automatically created by SolidWorks to URDF Exporter! Originally created by
-Stephen Brawner (brawner@gmail.com)
-     Commit Version: 1.6.0-4-g7f85cfe  Build Version: 1.6.7995.38578
-     For more information, please see http://wiki.ros.org/sw_urdf_exporter -->
 <robot xmlns:xacro="http://wiki.ros.org/xacro">
   <xacro:macro name="ar_gripper" params="
@@ -10,135 +6,83 @@
   ">
     <joint name="${tf_prefix}gripper_base_joint" type="fixed">
-      <origin xyz="0.0 0.0 0.0" rpy="-1.5708 0.0 0.0" />
-      <parent link="${parent}" />
-      <child link="${tf_prefix}gripper_base_link" />
+      <origin xyz="0.0 0.0 0.0" rpy="-1.5708 0.0 0.0"/>
+      <parent link="${parent}"/>
+      <child link="${tf_prefix}gripper_base_link"/>
     </joint>
     <link name="${tf_prefix}gripper_base_link">
-      <inertial>
-        <origin xyz="0.000218865638025569 -5.75810071732045E-05 0.0188189080442559" rpy="0 0 0" />
-        <mass value="0.0779213197542101" />
-        <inertia ixx="1.27018244320936E-05" ixy="-1.98293669536147E-07" ixz="-2.58632439119383E-07" iyy="2.84792796640278E-05" iyz="-4.25276765641554E-07" izz="3.57075748419373E-05" />
-      </inertial>
       <visual>
-        <origin xyz="0 0 0" rpy="0 0 0" />
         <geometry>
           <mesh filename="file://$(find annin_ar4_description)/meshes/ar4_gripper/gripper_base_link.stl" />
         </geometry>
         <material name="">
-          <color rgba="0.792156862745098 0.819607843137255 0.933333333333333 1" />
+          <color rgba="1 1 0 1"/>
         </material>
       </visual>
       <collision>
-        <origin xyz="0 0 0" rpy="0 0 0" />
         <geometry>
           <mesh filename="file://$(find annin_ar4_description)/meshes/ar4_gripper/gripper_base_link.stl" />
         </geometry>
       </collision>
+      <inertial>
+        <origin xyz="-0.00073621 -0.02341392 -0.00435302"/>
+        <mass value="0.08"/>
+        <inertia ixx="0.00002375" ixy="0.00000002" ixz="-0.00000017" iyy="0.00004082" iyz="-0.00000029" izz="0.00004254"/>
+      </inertial>
     </link>
     <link name="${tf_prefix}gripper_jaw1_link">
-      <inertial>
-        <origin xyz="0.0068393 0.0018263 -0.0052235" rpy="0 0 0" />
-        <mass value="0.0080032" />
-        <inertia ixx="7.6628E-07" ixy="2.1048E-07" ixz="4.3688E-09" iyy="1.0775E-06" iyz="-7.4587E-08" izz="1.3907E-06" />
-      </inertial>
       <visual>
-        <origin xyz="0 0 0" rpy="0 0 0" />
         <geometry>
           <mesh filename="file://$(find annin_ar4_description)/meshes/ar4_gripper/gripper_jaw1_link.stl" />
         </geometry>
         <material name="">
-          <color rgba="1 1 1 1" />
+          <color rgba="1 1 0 1"/>
         </material>
       </visual>
       <collision>
-        <origin xyz="0 0 0" rpy="0 0 0" />
         <geometry>
           <mesh filename="file://$(find annin_ar4_description)/meshes/ar4_gripper/gripper_jaw1_link.stl" />
         </geometry>
       </collision>
+      <inertial>
+        <origin xyz="-0.00435839 -0.00469536 0.00757141"/>
+        <mass value="0.01"/>
+        <inertia ixx="0.00000123" ixy="-0.00000004" ixz="0.00000012" iyy="0.00000115" iyz="0.00000016" izz="0.00000102"/>
+      </inertial>
     </link>
     <link name="${tf_prefix}gripper_jaw2_link">
-      <inertial>
-        <origin xyz="0.0068393 0.0018263 -0.0052235" rpy="0 0 0" />
-        <mass value="0.0080032" />
-        <inertia ixx="7.6628E-07" ixy="2.1048E-07" ixz="4.3688E-09" iyy="1.0775E-06" iyz="-7.4587E-08" izz="1.3907E-06" />
-      </inertial>
       <visual>
-        <origin xyz="-0.03 0 0.006" rpy="0 0 0" />
         <geometry>
           <mesh filename="file://$(find annin_ar4_description)/meshes/ar4_gripper/gripper_jaw2_link.stl" />
         </geometry>
         <material name="">
-          <color rgba="1 1 1 1" />
+          <color rgba="1 1 0 1"/>
         </material>
       </visual>
       <collision>
-        <origin xyz="-0.03 0 0.006" rpy="0 0 0" />
         <geometry>
           <mesh filename="file://$(find annin_ar4_description)/meshes/ar4_gripper/gripper_jaw2_link.stl" />
         </geometry>
       </collision>
+      <inertial>
+        <origin xyz="-0.00423971 -0.00491236 0.00814582"/>
+        <mass value="0.01"/>
+        <inertia ixx="0.00000118" ixy="-0.00000004" ixz="0.00000013" iyy="0.00000110" iyz="0.00000013" izz="0.00000101"/>
+      </inertial>
     </link>
     <joint name="${tf_prefix}gripper_jaw1_joint" type="prismatic">
-      <origin xyz="0.014 -0.0029 0.001" rpy="1.5708 0 0 " />
-      <parent link="${tf_prefix}gripper_base_link" />
-      <child link="${tf_prefix}gripper_jaw1_link" />
-      <axis xyz="-1 0 0" />
-      <limit lower="0" upper="0.015" effort="100" velocity="1.0" />
+      <origin xyz="0.0 -0.036 0" rpy="0.0 0.0 0.0"/>
+      <parent link="${tf_prefix}gripper_base_link"/>
+      <child link="${tf_prefix}gripper_jaw1_link"/>
+      <axis xyz="-1 0 0"/>
+      <limit lower="0" upper="0.014" effort="-1" velocity="1.0"/>
     </joint>
     <joint name="${tf_prefix}gripper_jaw2_joint" type="prismatic">
-      <origin xyz="0.014 0.0029 0.001" rpy="1.5708 0 0 " />
-      <parent link="${tf_prefix}gripper_base_link" />
-      <child link="${tf_prefix}gripper_jaw2_link" />
-      <axis xyz="1 0 0" />
-      <limit lower="0" upper="0.015" effort="100" velocity="1.0" />
+      <origin xyz="0.0 -0.036 0" rpy="0.0 ${-pi} 0.0"/>
+      <parent link="${tf_prefix}gripper_base_link"/>
+      <child link="${tf_prefix}gripper_jaw2_link"/>
+      <axis xyz="-1 0 0"/>
+      <limit lower="0" upper="0.014" effort="1000" velocity="1.0"/>
+      <mimic joint="${tf_prefix}gripper_jaw1_joint" multiplier="1" offset="0"/>
     </joint>
-    <!-- Gazebo friction properties for gripper jaws -->
-    <gazebo reference="${tf_prefix}gripper_jaw1_link">
-      <surface>
-        <friction>
-          <torsional>
-            <ode/>
-          </torsional>
-          <ode>
-            <mu>0.8</mu>
-            <mu2>0.8</mu2>
-            <slip1>0.001</slip1>
-            <slip2>0.001</slip2>
-          </ode>
-        </friction>
-        <contact>
-          <ode>
-            <max_vel>0.0</max_vel>
-            <min_depth>0.001</min_depth>
-            <kp>100000</kp>
-            <kd>1000</kd>
-          </ode>
-        </contact>
-      </surface>
-    </gazebo>
-    <gazebo reference="${tf_prefix}gripper_jaw2_link">
-      <surface>
-        <friction>
-          <torsional>
-            <ode/>
-          </torsional>
-          <ode>
-            <mu>0.8</mu>
-            <mu2>0.8</mu2>
-            <slip1>0.001</slip1>
-            <slip2>0.001</slip2>
-          </ode>
-        </friction>
-        <contact>
-          <ode>
-            <max_vel>0.0</max_vel>
-            <min_depth>0.001</min_depth>
-            <kp>100000</kp>
-            <kd>1000</kd>
-          </ode>
-        </contact>
-      </surface>
-    </gazebo>
   </xacro:macro>
 </robot>

File: annin_ar4_description/urdf/ar_macro.xacro (robot description, xacro)
@@ -65,5 +65,5 @@
         lower="${robot_parameters['j1_limit_min']}"
         upper="${robot_parameters['j1_limit_max']}"
-        effort="1000"
+        effort="-1"
         velocity="1.0472"
       />
@@ -99,5 +99,5 @@
         lower="${robot_parameters['j2_limit_min']}"
         upper="${robot_parameters['j2_limit_max']}"
-        effort="1000"
+        effort="-1"
         velocity="1.0472"
       />
@@ -133,5 +133,5 @@
         lower="${robot_parameters['j3_limit_min']}"
         upper="${robot_parameters['j3_limit_max']}"
-        effort="1000"
+        effort="-1"
         velocity="1.0472"
       />
@@ -167,5 +167,5 @@
         lower="${robot_parameters['j4_limit_min']}"
         upper="${robot_parameters['j4_limit_max']}"
-        effort="1000"
+        effort="-1"
         velocity="1.0472"
       />
@@ -194,5 +194,5 @@
     </link>
     <joint name="${tf_prefix}joint_5" type="revolute">
-      <origin rpy="${pi} 0 -1.57075" xyz="0 0 -0.22263"/>
+      <origin rpy="${pi} 0 -1.5708" xyz="0 0 -0.22263"/>
       <parent link="${tf_prefix}link_4"/>
       <child link="${tf_prefix}link_5"/>
@@ -201,5 +201,5 @@
         lower="${robot_parameters['j5_limit_min']}"
         upper="${robot_parameters['j5_limit_max']}"
-        effort="1000"
+        effort="-1"
         velocity="1.0472"
       />
@@ -235,5 +235,5 @@
         lower="${robot_parameters['j6_limit_min']}"
         upper="${robot_parameters['j6_limit_max']}"
-        effort="1000"
+        effort="-1"
         velocity="1.0472"
       />
@@ -246,10 +246,4 @@
       <origin xyz="0 0 0.0" rpy="0 0 0" />
     </joint>
-    <link name="${tf_prefix}laser_point" />
-    <joint name="${tf_prefix}laser_point_joint" type="fixed">
-      <parent link="${tf_prefix}ee_link" /> <!-- or laser_holder_link -->
-      <child link="${tf_prefix}laser_point" />
-      <origin xyz="0 0 0.106" rpy="0 0 0" /> <!-- Adjust if needed -->
-    </joint>
   </xacro:macro>
 </robot>

File: annin_ar4_driver/urdf/ar.urdf.xacro (robot description, xacro)
@@ -5,15 +5,14 @@
   <xacro:arg name="calibrate" default="True" />
   <xacro:arg name="tf_prefix" default="" />
-  <xacro:arg name="include_gripper" default="True" />
+  <xacro:arg name="include_gripper" default="true" />
   <xacro:include filename="$(find annin_ar4_description)/urdf/ar_macro.xacro" />
   <xacro:include filename="$(find annin_ar4_description)/urdf/ar.ros2_control.xacro" />
-  <xacro:include filename="$(find annin_ar4_description)/urdf/ar_gripper.ros2_control.xacro" />
-  <xacro:include filename="$(find annin_ar4_description)/urdf/ar_gripper_macro.xacro" />
   <link name="world" />
   <link name="ABB_base_link" />
-  <joint name="ABB_base_joint" type="fixed">
+  <joint name="ABB_base_link_to_world_joint" type="fixed">
     <parent link="world" />
     <child link="ABB_base_link" />
-    <origin xyz="0 -1.110  0" rpy="0 0 1.57079" />
+    <origin xyz="0 -1.110
+      0" rpy="0 0 1.57079" />
   </joint>
   <xacro:ar_robot
@@ -35,4 +34,6 @@
   />
   <xacro:if value="$(arg include_gripper)">
+    <xacro:include filename="$(find annin_ar4_description)/urdf/ar_gripper_macro.xacro" />
+    <xacro:include filename="$(find annin_ar4_description)/urdf/ar_gripper.ros2_control.xacro" />
     <xacro:ar_gripper
       tf_prefix="$(arg tf_prefix)"

File: annin_ar4_moveit_config/srdf/ar.srdf.xacro (robot description, xacro)
@@ -1,11 +1,11 @@
 <?xml version="1.0" encoding="UTF-8"?>
 <robot xmlns:xacro="http://wiki.ros.org/xacro" name="$(arg name)">
-  <xacro:arg name="include_gripper" default="true" />
+  <xacro:arg name="include_gripper" default="true"/>
   <xacro:arg name="tf_prefix" default="" />
-  <xacro:include filename="$(find annin_ar4_moveit_config)/srdf/ar_macro.srdf.xacro" />
-  <xacro:ar_srdf tf_prefix="$(arg tf_prefix)" />
+  <xacro:include filename="$(find annin_ar4_moveit_config)/srdf/ar_macro.srdf.xacro"/>
+  <xacro:ar_srdf tf_prefix="$(arg tf_prefix)"/>
   <xacro:if value="$(arg include_gripper)">
-    <xacro:include filename="$(find annin_ar4_moveit_config)/srdf/ar_gripper_macro.srdf.xacro" />
-    <xacro:ar_gripper_srdf tf_prefix="$(arg tf_prefix)" />
+    <xacro:include filename="$(find annin_ar4_moveit_config)/srdf/ar_gripper_macro.srdf.xacro"/>
+    <xacro:ar_gripper_srdf tf_prefix="$(arg tf_prefix)"/>
   </xacro:if>
 </robot>

File: annin_ar4_moveit_config/srdf/ar_gripper_macro.srdf.xacro (robot description, xacro)
@@ -1,7 +1,6 @@
-<?xml version="1.0"?>
+<?xml version="1.0" ?>
 <!--This does not replace URDF, and is not an extension of URDF.
     This is a format for representing semantic information about the robot structure.
-    A URDF file must exist for this robot as well, where the joints and the links that are referenced
-are defined
+    A URDF file must exist for this robot as well, where the joints and the links that are referenced are defined
 -->
 <robot xmlns:xacro="http://wiki.ros.org/xacro">
@@ -18,16 +17,11 @@
     </group_state>
     <group_state name="closed" group="ar_gripper">
-      <joint name="${tf_prefix}gripper_jaw1_joint" value="0" />
+      <joint name="${tf_prefix}gripper_jaw1_joint" value="0.000" />
     </group_state>
-    <disable_collisions link1="${tf_prefix}gripper_base_link" link2="${tf_prefix}gripper_jaw1_link"
-      reason="Adjacent" />
-    <disable_collisions link1="${tf_prefix}gripper_base_link" link2="${tf_prefix}gripper_jaw2_link"
-      reason="Adjacent" />
-    <disable_collisions link1="${tf_prefix}gripper_jaw1_link" link2="${tf_prefix}gripper_jaw2_link"
-      reason="Default" />
-    <disable_collisions link1="${tf_prefix}link_6" link2="${tf_prefix}gripper_base_link"
-      reason="Adjacent" />
-    <disable_collisions link1="${tf_prefix}link_5" link2="${tf_prefix}gripper_base_link"
-      reason="Adjacent" />
+    <disable_collisions link1="${tf_prefix}gripper_base_link" link2="${tf_prefix}gripper_jaw1_link" reason="Adjacent" />
+    <disable_collisions link1="${tf_prefix}gripper_base_link" link2="${tf_prefix}gripper_jaw2_link" reason="Adjacent" />
+    <disable_collisions link1="${tf_prefix}gripper_jaw1_link" link2="${tf_prefix}gripper_jaw2_link" reason="Default" />
+    <disable_collisions link1="${tf_prefix}link_6" link2="${tf_prefix}gripper_base_link" reason="Adjacent" />
+    <disable_collisions link1="${tf_prefix}link_5" link2="${tf_prefix}gripper_base_link" reason="Adjacent" />
   </xacro:macro>
 </robot>

File: annin_ar4_moveit_config/srdf/ar_macro.srdf.xacro (robot description, xacro)
@@ -1,7 +1,6 @@
-<?xml version="1.0"?>
+<?xml version="1.0" ?>
 <!--This does not replace URDF, and is not an extension of URDF.
     This is a format for representing semantic information about the robot structure.
-    A URDF file must exist for this robot as well, where the joints and the links that are referenced
-are defined
+    A URDF file must exist for this robot as well, where the joints and the links that are referenced are defined
 -->
 <robot xmlns:xacro="http://wiki.ros.org/xacro">
@@ -14,6 +13,5 @@
       <joint name="${tf_prefix}joint_5" />
       <joint name="${tf_prefix}joint_6" />
-      <joint name="${tf_prefix}ee_joint" />
-      <chain base_link="${tf_prefix}base_link" tip_link="${tf_prefix}ee_link" />
+      <joint name="${tf_prefix}ee_joint"/>
     </group>
     <group_state name="home" group="ar_manipulator">

File: annin_ar4_moveit_config/urdf/fake_ar.urdf.xacro (robot description, xacro)
@@ -1,8 +1,8 @@
 <?xml version="1.0"?>
 <robot xmlns:xacro="http://wiki.ros.org/xacro" name="$(arg ar_model)">
-  <xacro:include filename="$(find annin_ar4_description)/urdf/ar_macro.xacro" />
-  <xacro:include filename="$(find annin_ar4_description)/urdf/ar_gripper_macro.xacro" />
-  <xacro:include filename="$(find annin_ar4_description)/urdf/ar.ros2_control.xacro" />
-  <xacro:include filename="$(find annin_ar4_description)/urdf/ar_gripper.ros2_control.xacro" />
+  <xacro:include filename="$(find annin_ar4_description)/urdf/ar_macro.xacro"/>
+  <xacro:include filename="$(find annin_ar4_description)/urdf/ar_gripper_macro.xacro"/>
+  <xacro:include filename="$(find annin_ar4_description)/urdf/ar.ros2_control.xacro"/>
+  <xacro:include filename="$(find annin_ar4_description)/urdf/ar_gripper.ros2_control.xacro"/>
   <xacro:arg name="tf_prefix" default="" />
   <link name="world" />
