Commit message: jaw2 mimic: removed mimic on jaw2 for the AR4 and added control on jaw2

File: annin_ar4_description/urdf/ar_gripper.ros2_control.xacro (robot description, xacro)
@@ -30,6 +30,5 @@
       </joint>
       <joint name="${tf_prefix}gripper_jaw2_joint">
-        <param name="mimic">${tf_prefix}gripper_jaw1_joint</param>
-        <param name="multiplier">1</param>
+        <command_interface name="position" />
         <state_interface name="position">
           <param name="initial_value">0.0</param>

File: annin_ar4_moveit_config/srdf/ar_gripper_macro.srdf.xacro (robot description, xacro)
@@ -11,11 +11,13 @@
       <link name="${tf_prefix}gripper_jaw2_link" />
       <joint name="${tf_prefix}gripper_jaw1_joint" />
-      <passive_joint name="${tf_prefix}gripper_jaw2_joint" />
+      <joint name="${tf_prefix}gripper_jaw2_joint" />
     </group>
     <group_state name="closed" group="ar_gripper">
-      <joint name="${tf_prefix}gripper_jaw1_joint" value="0.014" />
+      <joint name="${tf_prefix}gripper_jaw1_joint" value="0.015" />
+      <joint name="${tf_prefix}gripper_jaw2_joint" value="0.015" />
     </group_state>
     <group_state name="open" group="ar_gripper">
       <joint name="${tf_prefix}gripper_jaw1_joint" value="0.000" />
+      <joint name="${tf_prefix}gripper_jaw2_joint" value="0.000" />
     </group_state>
     <disable_collisions link1="${tf_prefix}gripper_base_link" link2="${tf_prefix}gripper_jaw1_link" reason="Adjacent" />
