Commit message: gripper_fixed

File: annin_ar4_description/urdf/ar_gripper_macro.xacro (robot description, xacro)
@@ -65,5 +65,5 @@
       </inertial>
       <visual>
-        <origin xyz="0 0 0" rpy="0 0 0" />
+        <origin xyz="-0.03 0 0.006" rpy="0 0 0" />
         <geometry>
           <mesh filename="file://$(find annin_ar4_description)/meshes/ar4_gripper/gripper_jaw2_link.stl" />
@@ -74,5 +74,5 @@
       </visual>
       <collision>
-        <origin xyz="0 0 0" rpy="0 0 0" />
+        <origin xyz="-0.03 0 0.006" rpy="0 0 0" />
         <geometry>
           <mesh filename="file://$(find annin_ar4_description)/meshes/ar4_gripper/gripper_jaw2_link.stl" />
@@ -88,10 +88,9 @@
     </joint>
     <joint name="${tf_prefix}gripper_jaw2_joint" type="prismatic">
-      <origin xyz="-0.014 -0.0029 0.001" rpy="1.5708 0 0" />
+      <origin xyz="0.014 0.0029 0.001" rpy="1.5708 0 0 " />
       <parent link="${tf_prefix}gripper_base_link" />
       <child link="${tf_prefix}gripper_jaw2_link" />
       <axis xyz="1 0 0" />
       <limit lower="0" upper="0.015" effort="1000" velocity="1.0" />
-      <mimic joint="${tf_prefix}gripper_jaw1_joint" multiplier="1"/>
     </joint>
   </xacro:macro>

Commit message: ficxfriction_for_grasping_not_final (sebaey)

File: annin_ar4_description/urdf/ar_gripper_macro.xacro (robot description, xacro)
@@ -85,5 +85,5 @@
       <child link="${tf_prefix}gripper_jaw1_link" />
       <axis xyz="-1 0 0" />
-      <limit lower="0" upper="0.015" effort="1000" velocity="1.0" />
+      <limit lower="0" upper="0.015" effort="100" velocity="1.0" />
     </joint>
     <joint name="${tf_prefix}gripper_jaw2_joint" type="prismatic">
@@ -92,6 +92,49 @@
       <child link="${tf_prefix}gripper_jaw2_link" />
       <axis xyz="1 0 0" />
-      <limit lower="0" upper="0.015" effort="1000" velocity="1.0" />
+      <limit lower="0" upper="0.015" effort="100" velocity="1.0" />
     </joint>
+    <!-- Gazebo friction properties for gripper jaws -->
+    <gazebo reference="${tf_prefix}gripper_jaw1_link">
+      <surface>
+        <friction>
+          <torsional>
+            <ode/>
+          </torsional>
+          <ode>
+            <mu>2</mu>
+            <mu2>2</mu2>
+            <slip1>0.0001</slip1>
+            <slip2>0.0001</slip2>
+          </ode>
+        </friction>
+        <contact>
+          <ode>
+            <max_vel>0.0</max_vel>
+            <min_depth>0.001</min_depth>
+          </ode>
+        </contact>
+      </surface>
+    </gazebo>
+    <gazebo reference="${tf_prefix}gripper_jaw2_link">
+      <surface>
+        <friction>
+          <torsional>
+            <ode/>
+          </torsional>
+          <ode>
+            <mu>2</mu>
+            <mu2>2</mu2>
+            <slip1>0.0001</slip1>
+            <slip2>0.0001</slip2>
+          </ode>
+        </friction>
+        <contact>
+          <ode>
+            <max_vel>0.0</max_vel>
+            <min_depth>0.001</min_depth>
+          </ode>
+        </contact>
+      </surface>
+    </gazebo>
   </xacro:macro>
 </robot>

Commit message: AR4_gripper urdf: Adjusted origin values of joints and links for new gripper

File: annin_ar4_description/urdf/ar_gripper_macro.xacro (robot description, xacro)
@@ -6,26 +6,37 @@
   ">
     <joint name="${tf_prefix}gripper_base_joint" type="fixed">
-      <origin xyz="0.0 0.0 0.0" rpy="-1.5708 0.0 0.0"/>
-      <parent link="${parent}"/>
-      <child link="${tf_prefix}gripper_base_link"/>
+      <origin xyz="0.0 0.0 0.0" rpy="0.0 0.0 0.0" />
+      <parent link="${parent}" />
+      <child link="${tf_prefix}gripper_base_link" />
     </joint>
     <link name="${tf_prefix}gripper_base_link">
       <visual>
         <geometry>
-          <mesh filename="file://$(find annin_ar4_description)/meshes/ar4_gripper/gripper_base_link.stl" />
+          <mesh
+            filename="file://$(find annin_ar4_description)/meshes/ar4_gripper/gripper_base_link.STL" />
         </geometry>
         <material name="">
-          <color rgba="1 1 0 1"/>
+          <color rgba="1 1 0 1" />
         </material>
       </visual>
       <collision>
         <geometry>
-          <mesh filename="file://$(find annin_ar4_description)/meshes/ar4_gripper/gripper_base_link.stl" />
+          <mesh
+            filename="file://$(find annin_ar4_description)/meshes/ar4_gripper/gripper_base_link.STL" />
         </geometry>
       </collision>
       <inertial>
-        <origin xyz="-0.00073621 -0.02341392 -0.00435302"/>
-        <mass value="0.08"/>
-        <inertia ixx="0.00002375" ixy="0.00000002" ixz="-0.00000017" iyy="0.00004082" iyz="-0.00000029" izz="0.00004254"/>
+        <origin
+          xyz="0.000218865638025569 0.0025824189928268 0.0188189080442559"
+          rpy="0 0 0" />
+        <mass
+          value="0.0779213197542101" />
+        <inertia
+          ixx="1.27018244320936E-05"
+          ixy="-1.98293669536147E-07"
+          ixz="-2.58632439119383E-07"
+          iyy="2.84792796640278E-05"
+          iyz="-4.25276765641554E-07"
+          izz="3.57075748419373E-05" />
       </inertial>
     </link>
@@ -33,19 +44,30 @@
       <visual>
         <geometry>
-          <mesh filename="file://$(find annin_ar4_description)/meshes/ar4_gripper/gripper_jaw1_link.stl" />
+          <mesh
+            filename="file://$(find annin_ar4_description)/meshes/ar4_gripper/gripper_jaw1_link.STL" />
         </geometry>
         <material name="">
-          <color rgba="1 1 0 1"/>
+          <color rgba="1 1 0 1" />
         </material>
       </visual>
       <collision>
         <geometry>
-          <mesh filename="file://$(find annin_ar4_description)/meshes/ar4_gripper/gripper_jaw1_link.stl" />
+          <mesh
+            filename="file://$(find annin_ar4_description)/meshes/ar4_gripper/gripper_jaw1_link.STL" />
         </geometry>
       </collision>
       <inertial>
-        <origin xyz="-0.00435839 -0.00469536 0.00757141"/>
-        <mass value="0.01"/>
-        <inertia ixx="0.00000123" ixy="-0.00000004" ixz="0.00000012" iyy="0.00000115" iyz="0.00000016" izz="0.00000102"/>
+        <origin
+          xyz="-0.0031054 -0.0019355 0.0098549"
+          rpy="0 0 0" />
+        <mass
+          value="0.0066046" />
+        <inertia
+          ixx="1.5783E-06"
+          ixy="1.1866E-07"
+          ixz="1.5325E-07"
+          iyy="1.3594E-06"
+          iyz="-2.2561E-07"
+          izz="6.2333E-07" />
       </inertial>
     </link>
@@ -53,35 +75,38 @@
       <visual>
         <geometry>
-          <mesh filename="file://$(find annin_ar4_description)/meshes/ar4_gripper/gripper_jaw2_link.stl" />
+          <mesh
+            filename="file://$(find annin_ar4_description)/meshes/ar4_gripper/gripper_jaw2_link.STL" />
         </geometry>
         <material name="">
-          <color rgba="1 1 0 1"/>
+          <color rgba="1 1 0 1" />
         </material>
       </visual>
       <collision>
         <geometry>
-          <mesh filename="file://$(find annin_ar4_description)/meshes/ar4_gripper/gripper_jaw2_link.stl" />
+          <mesh
+            filename="file://$(find annin_ar4_description)/meshes/ar4_gripper/gripper_jaw2_link.STL" />
         </geometry>
       </collision>
       <inertial>
-        <origin xyz="-0.00423971 -0.00491236 0.00814582"/>
-        <mass value="0.01"/>
-        <inertia ixx="0.00000118" ixy="-0.00000004" ixz="0.00000013" iyy="0.00000110" iyz="0.00000013" izz="0.00000101"/>
+        <origin xyz="-0.00423971 -0.00491236 0.00814582" />
+        <mass value="0.01" />
+        <inertia ixx="0.00000118" ixy="-0.00000004" ixz="0.00000013" iyy="0.00000110"
+          iyz="0.00000013" izz="0.00000101" />
       </inertial>
     </link>
     <joint name="${tf_prefix}gripper_jaw1_joint" type="prismatic">
-      <origin xyz="0.0 -0.036 0" rpy="0.0 0.0 0.0"/>
-      <parent link="${tf_prefix}gripper_base_link"/>
-      <child link="${tf_prefix}gripper_jaw1_link"/>
-      <axis xyz="-1 0 0"/>
-      <limit lower="0" upper="0.014" effort="-1" velocity="1.0"/>
+      <origin xyz="0.0 -0.00026 0.0" rpy="0 0 0" />
+      <parent link="${tf_prefix}gripper_base_link" />
+      <child link="${tf_prefix}gripper_jaw1_link" />
+      <axis xyz="1 0 0" />
+      <limit lower="0" upper="0.014" effort="-1" velocity="1.0" />
     </joint>
     <joint name="${tf_prefix}gripper_jaw2_joint" type="prismatic">
-      <origin xyz="0.0 -0.036 0" rpy="0.0 ${-pi} 0.0"/>
-      <parent link="${tf_prefix}gripper_base_link"/>
-      <child link="${tf_prefix}gripper_jaw2_link"/>
-      <axis xyz="-1 0 0"/>
-      <limit lower="0" upper="0.014" effort="1000" velocity="1.0"/>
-      <mimic joint="${tf_prefix}gripper_jaw1_joint" multiplier="1" offset="0"/>
+      <origin xyz="0.0 -0.00026 0.0" rpy="0 0 0" />
+      <parent link="${tf_prefix}gripper_base_link" />
+      <child link="${tf_prefix}gripper_jaw2_link" />
+      <axis xyz="-1 0 0" />
+      <limit lower="0" upper="0.014" effort="1000" velocity="1.0" />
+      <mimic joint="${tf_prefix}gripper_jaw1_joint" multiplier="1" offset="0" />
     </joint>
   </xacro:macro>

Commit message: bye bye mimic joint

File: annin_ar4_description/urdf/ar_gripper_macro.xacro (robot description, xacro)
@@ -100,5 +100,5 @@
       <child link="${tf_prefix}gripper_jaw1_link" />
       <axis xyz="1 0 0" />
-      <limit lower="0" upper="0.014" effort="-1" velocity="1.0" />
+      <limit lower="0.0" upper="0.015" effort="100" velocity="1.0" />
     </joint>
     <joint name="${tf_prefix}gripper_jaw2_joint" type="prismatic">
@@ -107,7 +107,52 @@
       <child link="${tf_prefix}gripper_jaw2_link" />
       <axis xyz="-1 0 0" />
-      <limit lower="0" upper="0.014" effort="1000" velocity="1.0" />
-      <mimic joint="${tf_prefix}gripper_jaw1_joint" multiplier="1" offset="0" />
+      <limit lower="0.0" upper="0.015" effort="100" velocity="1.0" />
     </joint>
+    <gazebo reference="${tf_prefix}gripper_jaw1_link">
+      <surface>
+        <friction>
+          <torsional>
+            <ode/>
+          </torsional>
+          <ode>
+            <mu>0.8</mu>
+            <mu2>0.8</mu2>
+            <slip1>0.001</slip1>
+            <slip2>0.001</slip2>
+          </ode>
+        </friction>
+        <contact>
+          <ode>
+            <max_vel>0.0</max_vel>
+            <min_depth>0.001</min_depth>
+            <kp>100000</kp>
+            <kd>1000</kd>
+          </ode>
+        </contact>
+      </surface>
+    </gazebo>
+    <gazebo reference="${tf_prefix}gripper_jaw2_link">
+      <surface>
+        <friction>
+          <torsional>
+            <ode/>
+          </torsional>
+          <ode>
+            <mu>0.8</mu>
+            <mu2>0.8</mu2>
+            <slip1>0.001</slip1>
+            <slip2>0.001</slip2>
+          </ode>
+        </friction>
+        <contact>
+          <ode>
+            <max_vel>0.0</max_vel>
+            <min_depth>0.001</min_depth>
+            <kp>100000</kp>
+            <kd>1000</kd>
+          </ode>
+        </contact>
+      </surface>
+    </gazebo>
   </xacro:macro>
 </robot>

Commit message: gripper_physics + fix_grasp_deviation

File: annin_ar4_description/urdf/ar_gripper_macro.xacro (robot description, xacro)
@@ -52,7 +52,7 @@
       </visual>
       <collision>
+        <origin xyz="-0.024 0.0 0.065" rpy="0 0 0" />
         <geometry>
-          <mesh
-            filename="file://$(find annin_ar4_description)/meshes/ar4_gripper/gripper_jaw1_link.STL" />
+          <box size="0.007 0.018 0.035" />
         </geometry>
       </collision>
@@ -83,7 +83,7 @@
       </visual>
       <collision>
+        <origin xyz="0.024 0.0 0.065" rpy="0 0 0" />
         <geometry>
-          <mesh
-            filename="file://$(find annin_ar4_description)/meshes/ar4_gripper/gripper_jaw2_link.STL" />
+          <box size="0.007 0.018 0.035" />
         </geometry>
       </collision>
@@ -100,5 +100,5 @@
       <child link="${tf_prefix}gripper_jaw1_link" />
       <axis xyz="1 0 0" />
-      <limit lower="0.0" upper="0.015" effort="100" velocity="1.0" />
+      <limit lower="0.0" upper="0.015" effort="20" velocity="1.0" />
     </joint>
     <joint name="${tf_prefix}gripper_jaw2_joint" type="prismatic">
@@ -107,5 +107,5 @@
       <child link="${tf_prefix}gripper_jaw2_link" />
       <axis xyz="-1 0 0" />
-      <limit lower="0.0" upper="0.015" effort="100" velocity="1.0" />
+      <limit lower="0.0" upper="0.015" effort="20" velocity="1.0" />
     </joint>
     <gazebo reference="${tf_prefix}gripper_jaw1_link">
@@ -113,9 +113,13 @@
         <friction>
           <torsional>
-            <ode/>
+            <ode>
+              <coefficient>100.0</coefficient>
+              <use_patch_radius>true</use_patch_radius>
+              <patch_radius>0.015</patch_radius>
+            </ode>
           </torsional>
           <ode>
-            <mu>100</mu>
-            <mu2>100</mu2>
+            <mu>100.0</mu>
+            <mu2>100.0</mu2>
             <slip1>0.0</slip1>
             <slip2>0.0</slip2>
@@ -126,6 +130,6 @@
             <max_vel>0.0</max_vel>
             <min_depth>0.001</min_depth>
-            <kp>100000</kp>
-            <kd>10</kd>
+            <kp>1000000.0</kp>
+            <kd>1.0</kd>
           </ode>
         </contact>
@@ -136,9 +140,13 @@
         <friction>
           <torsional>
-            <ode/>
+            <ode>
+              <coefficient>100.0</coefficient>
+              <use_patch_radius>true</use_patch_radius>
+              <patch_radius>0.015</patch_radius>
+            </ode>
           </torsional>
           <ode>
-            <mu>100</mu>
-            <mu2>100</mu2>
+            <mu>100.0</mu>
+            <mu2>100.0</mu2>
             <slip1>0.0</slip1>
             <slip2>0.0</slip2>
@@ -149,6 +157,6 @@
             <max_vel>0.0</max_vel>
             <min_depth>0.001</min_depth>
-            <kp>100000</kp>
-            <kd>10</kd>
+            <kp>1000000.0</kp>
+            <kd>1.0</kd>
           </ode>
         </contact>
