Commit message: home position: set the home position for the robot where the gripper is facing downward.

File: annin_ar4_moveit_config/srdf/ar_macro.srdf.xacro (robot description, xacro)
@@ -22,5 +22,5 @@
       <joint name="${tf_prefix}joint_3" value="0" />
       <joint name="${tf_prefix}joint_4" value="0" />
-      <joint name="${tf_prefix}joint_5" value="0" />
+      <joint name="${tf_prefix}joint_5" value="1.57075" />
       <joint name="${tf_prefix}joint_6" value="0" />
     </group_state>

Commit message: AR4_home_position: adjust to be looking down as start position

File: annin_ar4_moveit_config/srdf/ar_macro.srdf.xacro (robot description, xacro)
@@ -22,5 +22,5 @@
       <joint name="${tf_prefix}joint_3" value="0" />
       <joint name="${tf_prefix}joint_4" value="0" />
-      <joint name="${tf_prefix}joint_5" value="1.57075" />
+      <joint name="${tf_prefix}joint_5" value="0" />
       <joint name="${tf_prefix}joint_6" value="0" />
     </group_state>
